Commit message: added a pendulum and changed plugin

File: robots/dreamer_ltw2.urdf (robot description, URDF)
Before this commit: robot dreamer, 47 links, 46 joints
Links:
- added link camera_linkL, mass 1e-5; visual box size=0.01 0.01 0.01
- added link camera_linkR, mass 1e-5; visual box size=0.01 0.01 0.01
Joints:
- added joint camera_jointL: type fixed, parent left_eye_yaw_link, child camera_linkL, origin xyz=0.02 0 0 rpy=0 0 0, axis 1 0 0
- added joint camera_jointR: type fixed, parent right_eye_yaw_link, child camera_linkR, origin xyz=0.02 0 0 rpy=0 0 0, axis 1 0 0
- joint left_eye_yaw: origin xyz=0 0.053 0 rpy=0 0 0 -> xyz=0 0.053 0 rpy=0 0 -0.152836
- joint right_eye_yaw: origin xyz=0 -0.053 0 rpy=0 0 0 -> xyz=0 -0.053 0 rpy=0 0 0.152836
